File: esp32.kicad_sch (KiCad schematic)
At the start: 24 parts, among them J5 TC2030-IDC, J6 Conn_01x08, J9 Conn_01x04, SW1 GT-TC029B-H025-L1N, SW2 GT-TC029B-H025-L1N, U11 RT9080-33GJ5, U12 ESP32-S3-WROOM-1, Y1 32.768kHz

Commit message: Nerdaxe Gamma
Parts:
- removed C21, C27, C49: 1uF, Capacitor_SMD:C_0402_1005Metric, symbol Device:C
- removed C30, C31: 6.8pF, Capacitor_SMD:C_0402_1005Metric, symbol Device:C
- removed C51: 10uF, Capacitor_SMD:C_0805_2012Metric, symbol Device:C
- removed C52: 0.1uF, Capacitor_SMD:C_0402_1005Metric, symbol Device:C
- removed D1: SS310, lcsc:SMA_L4.3-W2.6-LS5.2-RD, symbol lcsc:SS310_C85658
- removed J5: TC2030-IDC, Connector:Tag-Connect_TC2030-IDC-NL_2x03_P1.27mm_Vertical, symbol Espressif:TC2030-IDC-NL
- removed J6: Conn_01x08, Connector_PinHeader_2.54mm:PinHeader_1x07_P2.54mm_Vertical, symbol Connector_Generic:Conn_01x07
- removed J9: Conn_01x04, Connector_PinHeader_2.54mm:PinHeader_1x04_P2.54mm_Vertical, symbol Connector_Generic:Conn_01x04
- removed R1: 10k, Resistor_SMD:R_0402_1005Metric, symbol Device:R_US
- removed SW1, SW2: GT-TC029B-H025-L1N, bitaxe:SW_CS1213AGF260_CRS, symbol lcsc:GT-TC029B-H025-L1N
- removed TP17, TP18, TP19, TP22, TP23, TP31: TestPoint, TestPoint:TestPoint_Pad_D1.5mm, symbol Connector:TestPoint
- removed U11: RT9080-33GJ5, bitaxe:RT9080-33GJ5, symbol bitaxe:RT9080-33GJ5
- removed U12: ESP32-S3-WROOM-1, Espressif:ESP32-S3-WROOM-1, symbol Espressif:ESP32-S3-WROOM-1
- removed USB1: 10118193-0001LF, bitaxe:USB_10118193-0001LF_AMP, symbol lcsc:U254-051T-4BHJ25-F2S
- removed Y1: 32.768kHz, bitaxe:SC32S-7PF20PPM, symbol Device:Crystal
- added D2: US1D, Diode_SMD:D_SMA, symbol Diode:US1D
- added U11: T-Display-S3, bitaxe:T-Display-S3, symbol bitaxe:T-Display-S3
Connections:
- net 3V3: now also U11.1 (3V), U11.13 (3V)
- net 5V: now also D2.2 (A)
- net GND: now also U11.11 (GND), U11.14 (GND), U11.15 (GND), U11.23 (GND), U11.24 (GND)
- net PGOOD: now also U11.6 (GPIO11)
- net RST: now also U11.2 (GPIO1)
- net RX: now also U11.20 (GPIO18)
- net SCL: now also U11.22 (GPIO43)
- net SDA: now also U11.21 (GPIO44)
- net TX: now also U11.19 (GPIO17)
- net VDD: now also U11.3 (GPIO2)
- new net: D2.1 (K), U11.12 (5V)
- new net SMB_ALRT: U11.8 (GPIO13)
Other:
- note added: "Nerdaxe gamma"
- note removed: "3V3 Debug Header"
- note removed: "ESP32 3V3 LDO"
- note removed: "OLED Display Header"
- note removed: "Program the ESP32 with a ESP-PROG and a Tag Connect TC2030-IDC"
- note removed: "RTC Clock Crystal"
- note removed: "SSD1306 128x32 I2C OLED"
- title: le bitaxeTTGO -> bitaxeGamma
