File: fan.kicad_sch (KiCad schematic)
At the start: 9 parts, among them J4 Conn_01x04, U7 EMC2101

Commit message: Nerdaxe Gamma
Parts:
- removed C28: 220uF, Capacitor_SMD:CP_Elec_6.3x7.7, symbol Device:C_Polarized
- added C50: 470pF, Capacitor_SMD:C_0402_1005Metric, symbol Device:C
- added C51: 47uF, Capacitor_SMD:C_1210_3225Metric, symbol Device:C
- added R22, R23: 100, Resistor_SMD:R_0402_1005Metric, symbol DayMiner-eagle-import:RESISTOR0402-RES
- added TP35, TP36: TestPoint, TestPoint:TestPoint_Pad_D1.5mm, symbol Connector:TestPoint
- C52: renamed from C29; DK 1292-1639-1-ND -> 1276-1234-1-ND; LCSC Part C1525 -> (none); PARTNO 0402X104K100CT -> CL05A104KO5NNNC
- C53: renamed from C33; DK 1292-1639-1-ND -> 1276-1234-1-ND; LCSC Part C1525 -> (none); PARTNO 0402X104K100CT -> CL05A104KO5NNNC
- R25: renamed from R9; LCSC Part C269674 -> (none)
- R51: LCSC Part C365033 -> (none)
- U10: renamed from U7; symbol dayminer:EMC2101 -> bitaxe:EMC2101
- renumbered J4 to J6, TP16 to TP37, TP15 to TP38
Connections:
- net 3V3: no longer C53.1, R25.2
- net 5V: now also C53.1, R25.2, C51.1
- net GND: now also C51.2
- net TEMP_DP: now reaches U10.2 (DP)
- net TEMP_DP: now also C50.1, R23.2
- net TEMP_DN: now reaches U10.3 (DN)
- net TEMP_DN: now also C50.2, R22.1
- new net TEMP_N: R22.2, TP36.1
- new net TEMP_P: R23.1, TP35.1
Other:
- note added: "Nerdaxe gamma"
- title: NerdAxe -> bitaxeGamma
- moved on the sheet: J6, R51, TP37, TP38, U10
