File: power.kicad_sch (KiCad schematic)
At the start: 29 parts, among them Q1 CSD17311Q5, Q2 CSD17311Q5, Q3 2N7002K, U10 DS4432U+, U8 INA260, U9 TPS40305

Commit message: Nerdaxe Gamma
Parts:
- removed C34, C36, C37: 47uF, Capacitor_SMD:C_1210_3225Metric, symbol Device:C
- removed C35, C44: 1uF, Capacitor_SMD:C_0402_1005Metric, symbol Device:C
- removed C38: 1uF, Capacitor_SMD:C_0805_2012Metric, symbol Device:C
- removed C39: 3.3nF, Capacitor_SMD:C_0402_1005Metric, symbol Device:C
- removed C40: 180pF, Capacitor_SMD:C_0805_2012Metric, symbol Device:C
- removed C41: 1.5nF, Capacitor_SMD:C_0805_2012Metric, symbol Device:C
- removed C42: 0.1uF, Capacitor_SMD:C_0402_1005Metric, symbol Device:C
- removed C43: 10uF, Capacitor_SMD:C_0805_2012Metric, symbol Device:C
- removed C45: 470pF, Capacitor_SMD:C_0805_2012Metric, symbol Device:C
- removed C46: 220uF, TPS40305_supply:CAP_2R5TPE220MAFB, symbol Device:C_Polarized
- removed C47: 100uF, Capacitor_SMD:C_1206_3216Metric, symbol Device:C
- removed Q1, Q2: CSD17311Q5, TPS40305_supply:CSD17311Q5, symbol TPS40305:Q_NMOS_CSD17311Q5
- removed Q3: 2N7002K, Package_TO_SOT_SMD:SOT-323_SC-70, symbol Transistor_FET:2N7002K
- removed R16: 80k, Resistor_SMD:R_0402_1005Metric, symbol Device:R_US
- removed R17: DNP, Resistor_SMD:R_0402_1005Metric, symbol Device:R_US
- removed U10: DS4432U+, Package_SO:TSSOP-8_3x3mm_P0.65mm, symbol TPS40305:DS4432U+
- removed U8: INA260, Package_SO:TSSOP-16_4.4x5mm_P0.65mm, symbol Sensor:INA260
- removed U9: TPS40305, TPS40305_supply:TPS40305, symbol TPS40305:TPS40305
- added C1, C5, C7: 1uF, Capacitor_SMD:C_0402_1005Metric, symbol Device:C
- added C10: 4.7uF, Capacitor_SMD:C_0402_1005Metric, symbol Device:C
- added C11: 1000pF, Capacitor_SMD:C_0805_2012Metric, symbol Device:C
- added C12, C8: 0.1uF, Capacitor_SMD:C_0402_1005Metric, symbol Device:C
- added C13: 100pF, Capacitor_SMD:C_0402_1005Metric, symbol Device:C
- added C14, C15, C16: 22uF, Capacitor_SMD:C_0805_2012Metric, symbol Device:C
- added C17, C18, C19, C20: 100uF, Capacitor_SMD:C_1206_3216Metric, symbol Device:C
- added C2: 10uF, Capacitor_SMD:C_0805_2012Metric, symbol Device:C
- added C3, C4: 47uF, Capacitor_SMD:C_1210_3225Metric, symbol Device:C
- added C6: 4700pF, Capacitor_SMD:C_0402_1005Metric, symbol Device:C
- added C9: 2200pF, Capacitor_SMD:C_0402_1005Metric, symbol Device:C
- added D1: SMAJ5.0A, Diode_SMD:D_SMA, symbol Diode:SMAJ5.0A
- added R1: 8.25k, Resistor_SMD:R_0402_1005Metric, symbol Device:R_US
- added R11: 10, Resistor_SMD:R_0402_1005Metric, symbol Device:R_US
- added R2, R3, R7: ~, Resistor_SMD:R_0402_1005Metric, symbol Device:R_US
- added R5: 14.7k, Resistor_SMD:R_0402_1005Metric, symbol Device:R_US
- added R6: 0, Resistor_SMD:R_0402_1005Metric, symbol Device:R_US
- added R8: 3.74k, Resistor_SMD:R_0402_1005Metric, symbol Device:R_US
- added R9: 11.8k, Resistor_SMD:R_0402_1005Metric, symbol Device:R_US
- added T1: net-tie, bitaxe:NetTie-0.25mm, symbol bitaxe:net-tie
- added TP3, TP4: TestPoint, TestPoint:TestPoint_Pad_D1.5mm, symbol Connector:TestPoint
- added U2: TPS546D24ARVFR, bitaxe:LQFN40-CLIP, symbol bitaxe:TPS546D24
- L1: value 150nH -> 300nH; footprint TPS40305_supply:FP1005R1-R15-R -> bitaxe:SLC1175-271MEC_COC; DK 513-1568-1-ND -> (none); Mouser (none) -> 994-SLC1175-271MEC; PARTNO FP1005R1-R15-R -> SLC1175-301MEC
- R10: value 3.83k -> 68.1k; DK 311-3.83KLRCT-ND -> YAG3213CT-ND; LCSC Part C100402 -> (none); PARTNO RC0402FR-073K83L -> RC0402FR-0768K1L
- R12: value 4.12k -> 1; footprint Resistor_SMD:R_0402_1005Metric -> Resistor_SMD:R_1206_3216Metric; DK RMCF0402FT4K12CT-ND -> CSR1206FT1R00CT-ND; LCSC Part C327340 -> (none); PARTNO RMCF0402FT4K12 -> CSR1206FT1R00
- R13: value 1.33k -> 49.9; DK 311-1.33KLRCT-ND -> 311-49.9LRCT-ND; LCSC Part C334646 -> (none); PARTNO RC0402FR-071K33L -> RC0402FR-0749R9L
- R14: value 4.99k -> 49.9; DK 311-4.99KLRCT-ND -> 311-49.9LRCT-ND; LCSC Part C140155 -> (none); PARTNO RC0402FR-074K99L -> RC0402FR-0749R9L
- R15: value 3.32k -> 10k; DK 311-3.32KLRCT-ND -> 311-10KJRCT-ND; LCSC Part C284517 -> (none); PARTNO RC0402FR-073K32L -> RC0402JR-0710KL
- R4: value 10k -> ~; DK 311-10KJRCT-ND -> (none); LCSC Part C269674 -> (none); PARTNO RC0402JR-0710KL -> (none); now not fitted; now left out of the parts list
Connections:
- net 3V3: now also R15.2; no longer R4.1
- net 5V: now also C2.1, C3.1, C4.1, C6.1, C7.1, C9.1, D1.1 (A1), R11.1, R9.1, U2.21 (PVIN), U2.22 (PVIN), U2.23 (PVIN), U2.24 (PVIN), U2.25 (PVIN)
- net GND: now also R12.1, R13.2, C10.2, C14.2, C15.2, C16.2, C17.2, C18.2, C19.2, C2.2, C20.2, C3.2, C4.2, C6.2, C7.2, C9.2, D1.2 (A2), T1.2, TP4.1, U2.13 (PGND), U2.14 (PGND), U2.15 (PGND), U2.16 (PGND), U2.17 (PGND), U2.18 (PGND), U2.19 (PGND), U2.20 (PGND), U2.41 (PAD); no longer R12.2, R15.2
- net PGOOD: now also R15.1, U2.1 (PGD); no longer R4.2
- net SCL: now also U2.3 (PMB_CLK)
- net SDA: now also U2.2 (PMB_DATA)
- net SW: now also C11.2, C12.2, U2.10 (SW), U2.11 (SW), U2.12 (SW), U2.8 (SW), U2.9 (SW)
- net VOUT: now also C14.1, C15.1, C16.1, C17.1, C18.1, C19.1, C20.1, TP3.1; no longer R13.1
- net at R10.1: now also R4.2, U2.30 (VSEL)
- removed net OUT0: R10.2, R14.2, R15.1
- new net: C13.1, R14.2, U2.33 (VOSNS)
- new net: C10.1, U2.28 (VDD5)
- new net: C1.1, U2.5 (DRTN)
- new net: C1.2, R1.1, R2.1, R3.1, R4.1, U2.4 (BP1V5)
- new net: C8.1, R8.1, R9.2, U2.27 (EN/UVLO)
- new net: C13.2, R13.1, U2.34 (GOSNS)
- new net: C5.2, R11.2, U2.26 (AVIN)
- new net: R2.2, R6.1, U2.29 (MSEL2)
- new net: R3.2, R7.1, U2.31 (ADRSEL)
- new net: R1.2, R5.2, U2.32 (MSEL1)
- new net: C12.1, U2.7 (BOOT)
- new net: C11.1, R12.2
- new net AGND: C5.1, C8.2, R10.2, R5.1, R6.2, R7.2, R8.2, T1.1, U2.37 (AGND)
- new net SMB_ALRT: U2.6 (SMB_ALRT)
- no-connect marks 0 -> 5
Other:
- note added: "Connect at U3 Pin 37"
- note added: "I2C ADDR = 0x24"
- note added: "Input 4.5-5.5V"
- note added: "Output 1.2V nominal 20A max"
- note added: "PGD is an open drain output from the TPS546D24. Pull up to 3.3V"
- note added: "TPS546D24A is a Buck regulator that steps 4.5-5.5V down to 1.2V @ 20A for the BM1368"
- note added: "https://webench.ti.com/appinfo/webench/scripts/SDP.cgi?ID=3808DBEB40D18F5D"
- note removed: "DS4432U+ Lets us change the TPS40305 voltage over I2C"
- note removed: "I2C Address: 0x40"
- note removed: "I2C Address: 0x48"
- note removed: "Power Monitor"
- note removed: "TPS40305 is a Buck regulator that steps 5V down to around 1.5V for the BM1397"
- note removed: "The INA260 is currently out of stock everywhere. This part is totally optional, feel free to leave it out if you can't source it. If you DNP it, close J7"
- note removed: "Vfb = 0.6V"
- title: NerdAxe -> bitaxeGamma
